Commit message: [feat] - init commit with velodyne lidar on hector quadrotot

File: hector_quadrotor/hector_quadrotor_description/urdf/quadrotor_base.urdf.xacro (robot description, xacro)
@@ -29,3 +29,8 @@
     </xacro:sonar_sensor>
   </xacro:macro>
+    <!-- Velodyne -->
+    <xacro:include filename="$(find hector_sensors_description)/urdf/velodyne_vlp16.urdf.xacro" />
+    <xacro:velodyne_vlp16 name="velodyne" parent="base_link">
+      <origin xyz="0.0 0.0 0.03585" rpy="0 0 0"/>
+    </xacro:velodyne_vlp16>
 </robot>

File: hector_quadrotor/hector_quadrotor_gazebo/urdf/quadrotor_sensors.gazebo.xacro (robot description, xacro)
@@ -55,4 +55,14 @@
             <frameName>$(arg world_frame)</frameName>
           </plugin>
+          <plugin filename="libgazebo_ros_p3d.so" name="p3d_base_controller">
+            <alwaysOn>true</alwaysOn>
+            <updateRate>10.0</updateRate>
+            <bodyName>base_link</bodyName>
+            <topicName>platform/ground_truth_odometry</topicName>
+            <gaussianNoise>0.01</gaussianNoise>
+            <frameName>world</frameName>
+            <xyzOffsets>0 0 0</xyzOffsets>
+            <rpyOffsets>0 0 0</rpyOffsets>
+    </plugin>
         </gazebo>
   </xacro:macro>
